File: hardware/main/sd-card-mux.kicad_sch (KiCad schematic)
At the start: 80 parts, among them J1 1050170001, J2 NPTC081KFXC-RC, J3 687108183722, J4 Micro-SD, J5 Conn_01x08_Male, SW1 JS102011SCQN, SW2 DS04-254-2-01BK-SMT, U1 AT24CS02-SSHM, U10 SN74LVC2G157, U2 USB2640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

Commit message: Added breakout board and documentation.
Other:
- title: (none) -> SD-Card-MUX
Changed lines of the file:
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@@
 (kicad_sch (version 20211123) (generator eeschema)
   (paper "B")
+  (title_block
+    (title "SD-Card-MUX")
+    (comment 1 "License: GPL-3.0")
+  )
   (junction (at 52.07 31.75) (diameter 0) (color 0 0 0 0)
   )
