File: hardware/microsd-breakout/microsd-breakout.kicad_pcb (KiCad board)
At the start: 2 copper layers, 11 x 20 mm, 5 parts, among them J1 687108183722, J2 Conn_01x08_Male

Commit message: Added breakout board and documentation.
Parts:
- removed the REF** at (171.2, 84.0)
- removed the REF** at (159.3, 84.0)
- removed the REF** at (165.3, 89.7)
- added REF**: Tab, kikit:Tab, F.Cu at (170.8, 73.9)
- added REF**: Tab, kikit:Tab, F.Cu at (166.0, 69.0)
- added REF**: Tab, kikit:Tab, F.Cu at (170.8, 83.0)
- added REF1: Tab, kikit:Tab, F.Cu at (165.3, 89.2)
Changed lines of the file:
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@@
   (net 10 "unconnected-(J1-Pad10)")
   (footprint "kikit:Tab" (layer "F.Cu")
-    (at 171.25 84 180)
+    (at 165.3 89.2 90)
+    (descr "A symbol representing annotation for tab placement")
+    (attr exclude_from_pos_files exclude_from_bom)
+    (fp_text reference "REF1" (at 0 -2 90) (layer "F.SilkS") hide
+      (effects (font (size 1 1) (thickness 0.15)))
+    )
+    (fp_text value "Tab" (at -2.75 -1 90) (layer "Dwgs.User")
+      (effects (font (size 1.2 1.2) (thickness 0.2)))
+    )
+    (fp_text user "KIKIT: width: 3mm" (at -5.5 0) (layer "Dwgs.User")
+      (effects (font (size 1 1) (thickness 0.15)))
+    )
+    (fp_line (start 0.25 0) (end -2.75 0) (layer "Dwgs.User") (width 0.3))
+    (fp_line (start 0.25 1) (end 0.25 -1) (layer "Dwgs.User") (width 0.3))
+    (fp_line (start 0.25 0) (end -0.75 -1) (layer "Dwgs.User") (width 0.3))
+    (fp_line (start 0.25 0) (end -0.75 1) (layer "Dwgs.User") (width 0.3))
+  )
+  (footprint "kikit:Tab" (layer "F.Cu")
+    (at 170.8 73.9 180)
     (descr "A symbol representing annotation for tab placement")
     (attr exclude_from_pos_files exclude_from_bom)
@@
       (effects (font (size 1 1) (thickness 0.15)))
     )
-    (fp_line (start 0.25 0) (end -0.75 1) (layer "Dwgs.User") (width 0.3))
     (fp_line (start 0.25 1) (end 0.25 -1) (layer "Dwgs.User") (width 0.3))
+    (fp_line (start 0.25 0) (end -0.75 -1) (layer "Dwgs.User") (width 0.3))
     (fp_line (start 0.25 0) (end -2.75 0) (layer "Dwgs.User") (width 0.3))
-    (fp_line (start 0.25 0) (end -0.75 -1) (layer "Dwgs.User") (width 0.3))
-  )
-  (footprint "kikit:Tab" (layer "F.Cu")
-    (at 159.35 84)
-    (descr "A symbol representing annotation for tab placement")
-    (attr exclude_from_pos_files exclude_from_bom)
-    (fp_text reference "REF**" (at 0 -2) (layer "F.SilkS") hide
-      (effects (font (size 1 1) (thickness 0.15)))
-    )
-    (fp_text value "Tab" (at -2.75 -1) (layer "Dwgs.User")
-      (effects (font (size 1.2 1.2) (thickness 0.2)))
-    )
-    (fp_text user "KIKIT: width: 3mm" (at -5.5 0 90) (layer "Dwgs.User")
-      (effects (font (size 1 1) (thickness 0.15)))
-    )
-    (fp_line (start 0.25 0) (end -0.75 1) (layer "Dwgs.User") (width 0.3))
-    (fp_line (start 0.25 0) (end -0.75 -1) (layer "Dwgs.User") (width 0.3))
-    (fp_line (start 0.25 1) (end 0.25 -1) (layer "Dwgs.User") (width 0.3))
-    (fp_line (start 0.25 0) (end -2.75 0) (layer "Dwgs.User") (width 0.3))
-  )
-  (footprint "kikit:Tab" (layer "F.Cu")
-    (at 165.3 89.7 90)
-    (descr "A symbol representing annotation for tab placement")
-    (attr exclude_from_pos_files exclude_from_bom)
-    (fp_text reference "REF**" (at 0 -2 90) (layer "F.SilkS") hide
-      (effects (font (size 1 1) (thickness 0.15)))
-    )
-    (fp_text value "Tab" (at -2.75 -1 90) (layer "Dwgs.User")
-      (effects (font (size 1.2 1.2) (thickness 0.2)))
-    )
-    (fp_text user "KIKIT: width: 3mm" (at -5.5 0) (layer "Dwgs.User")
-      (effects (font (size 1 1) (thickness 0.15)))
-    )
-    (fp_line (start 0.25 0) (end -2.75 0) (layer "Dwgs.User") (width 0.3))
-    (fp_line (start 0.25 0) (end -0.75 -1) (layer "Dwgs.User") (width 0.3))
-    (fp_line (start 0.25 1) (end 0.25 -1) (layer "Dwgs.User") (width 0.3))
     (fp_line (start 0.25 0) (end -0.75 1) (layer "Dwgs.User") (width 0.3))
   )
@@
       (net 8 "/DAT1") (pinfunction "Pin_8") (pintype "passive"))
   )
+  (footprint "kikit:Tab" (layer "F.Cu")
+    (at 165.96 69.05 -90)
+    (descr "A symbol representing annotation for tab placement")
+    (attr exclude_from_pos_files exclude_from_bom)
+    (fp_text reference "REF**" (at 0 -2 90) (layer "F.SilkS") hide
+      (effects (font (size 1 1) (thickness 0.15)))
+    )
+    (fp_text value "Tab" (at -2.75 -1 90) (layer "Dwgs.User")
+      (effects (font (size 1.2 1.2) (thickness 0.2)))
+    )
+    (fp_text user "KIKIT: width: 3mm" (at -5.5 0) (layer "Dwgs.User")
+      (effects (font (size 1 1) (thickness 0.15)))
+    )
+    (fp_line (start 0.25 0) (end -2.75 0) (layer "Dwgs.User") (width 0.3))
+    (fp_line (start 0.25 1) (end 0.25 -1) (layer "Dwgs.User") (width 0.3))
+    (fp_line (start 0.25 0) (end -0.75 -1) (layer "Dwgs.User") (width 0.3))
+    (fp_line (start 0.25 0) (end -0.75 1) (layer "Dwgs.User") (width 0.3))
+  )
+  (footprint "kikit:Tab" (layer "F.Cu")
+    (at 170.8 83 180)
+    (descr "A symbol representing annotation for tab placement")
+    (attr exclude_from_pos_files exclude_from_bom)
+    (fp_text reference "REF**" (at 0 -2) (layer "F.SilkS") hide
+      (effects (font (size 1 1) (thickness 0.15)))
+    )
+    (fp_text value "Tab" (at -2.75 -1) (layer "Dwgs.User")
+      (effects (font (size 1.2 1.2) (thickness 0.2)))
+    )
+    (fp_text user "KIKIT: width: 3mm" (at -5.5 0 90) (layer "Dwgs.User")
+      (effects (font (size 1 1) (thickness 0.15)))
+    )
+    (fp_line (start 0.25 1) (end 0.25 -1) (layer "Dwgs.User") (width 0.3))
+    (fp_line (start 0.25 0) (end -0.75 -1) (layer "Dwgs.User") (width 0.3))
+    (fp_line (start 0.25 0) (end -2.75 0) (layer "Dwgs.User") (width 0.3))
+    (fp_line (start 0.25 0) (end -0.75 1) (layer "Dwgs.User") (width 0.3))
+  )
   (footprint "sd-card-mux:Wurth_FPC_687108183722" (layer "B.Cu")
